Commit message: Auto stash before merge of "master" and "origin/master"
3D Models Added

File: urdf/example.urdf.xacro (robot description, xacro)
@@ -6,4 +6,4 @@
   name="sick_tim">
   <xacro:include filename="$(find sick_scan)/urdf/sick_scan.urdf.xacro" />
-  <xacro:sick_tim310 name="laser" ros_topic="scan" />
+  <xacro:sick_tim_5xx name="laser" ros_topic="scan" />
 </robot>

File: urdf/sick_scan.urdf.xacro (robot description, xacro)
@@ -4,9 +4,9 @@
   xmlns:sensor="http://playerstage.sourceforge.net/gazebo/xmlschema/#sensor"
   xmlns:xacro="http://ros.org/wiki/xacro">
-  <xacro:macro name="sick_tim310" params="name ros_topic">
+  <xacro:macro name="sick_tim_3xx" params="name ros_topic">
     <xacro:sick_scan name="${name}" ros_topic="${ros_topic}"
       length="0.06" width="0.06" height="0.079" mass="0.150" z_offset="0.05595"
       min_range="0.05" max_range="4.0"
-      mesh="package://sick_scan/meshes/sick_tim310.stl" />
+      mesh="package://sick_scan/meshes/sick_tim_3xx.stl" />
   </xacro:macro>
   <xacro:macro name="sick_tim_5xx" params="name ros_topic">
@@ -14,11 +14,11 @@
       length="0.06" width="0.06" height="0.086" mass="0.250" z_offset="0.06296"
       min_range="0.05" max_range="10.0"
-      mesh="package://sick_scan/meshes/sick_tim551.stl" />
+      mesh="package://sick_scan/meshes/sick_tim_5xx.stl" />
   </xacro:macro>
-  <xacro:macro name="sick_mrs_1000" params="name ros_topic">
+  <xacro:macro name="sick_mrs_1xxx" params="name ros_topic">
     <xacro:sick_scan name="${name}" ros_topic="${ros_topic}"
       length="0.1519" width="0.15" height="0.0926" mass="0.250" z_offset="0.0658"
       min_range="0.05" max_range="10.0"
-      mesh="package://sick_scan/meshes/sick_MRS1000.stl" />
+      mesh="package://sick_scan/meshes/sick_mrs_1xxx.stl" />
   </xacro:macro>
   <xacro:macro name="sick_scan" params="name ros_topic length width height mass z_offset min_range max_range mesh">

Commit message: Auto stash before merge of "master" and "origin/master"
2D Model for tim_5xx added and launchfiles renamed

File: urdf/example.urdf.xacro (robot description, xacro)
@@ -4,6 +4,7 @@
   xmlns:sensor="http://playerstage.sourceforge.net/gazebo/xmlschema/#sensor"
   xmlns:xacro="http://ros.org/wiki/xacro"
-  name="sick_tim">
+  name="sick_scan">
   <xacro:include filename="$(find sick_scan)/urdf/sick_scan.urdf.xacro" />
   <xacro:sick_tim_5xx name="laser" ros_topic="scan" />
+  <xacro:sick_mrs_1xxx name="laser" ros_topic="scan" />
 </robot>

File: urdf/sick_scan.urdf.xacro (robot description, xacro)
@@ -4,23 +4,17 @@
   xmlns:sensor="http://playerstage.sourceforge.net/gazebo/xmlschema/#sensor"
   xmlns:xacro="http://ros.org/wiki/xacro">
-  <xacro:macro name="sick_tim_3xx" params="name ros_topic">
-    <xacro:sick_scan name="${name}" ros_topic="${ros_topic}"
+  <xacro:macro name="sick_tim_5xx" params="name ros_topic">
+    <xacro:sick_tim name="${name}" ros_topic="${ros_topic}"
       length="0.06" width="0.06" height="0.079" mass="0.150" z_offset="0.05595"
       min_range="0.05" max_range="4.0"
-      mesh="package://sick_scan/meshes/sick_tim_3xx.stl" />
-  </xacro:macro>
-  <xacro:macro name="sick_tim_5xx" params="name ros_topic">
-    <xacro:sick_scan name="${name}" ros_topic="${ros_topic}"
-      length="0.06" width="0.06" height="0.086" mass="0.250" z_offset="0.06296"
-      min_range="0.05" max_range="10.0"
       mesh="package://sick_scan/meshes/sick_tim_5xx.stl" />
   </xacro:macro>
   <xacro:macro name="sick_mrs_1xxx" params="name ros_topic">
-    <xacro:sick_scan name="${name}" ros_topic="${ros_topic}"
-      length="0.1519" width="0.15" height="0.0926" mass="0.250" z_offset="0.0658"
-      min_range="0.05" max_range="10.0"
-      mesh="package://sick_scan/meshes/sick_mrs_1xxx.stl" />
+    <xacro:sick_tim name="${name}" ros_topic="${ros_topic}"
+      length="0.06" width="0.06" height="0.079" mass="0.150" z_offset="0.05595"
+      min_range="0.05" max_range="4.0"
+      mesh="package://sick_scan/meshes/sick_tim_5xx.stl" />
   </xacro:macro>
-  <xacro:macro name="sick_scan" params="name ros_topic length width height mass z_offset min_range max_range mesh">
+  <xacro:macro name="sick_tim" params="name ros_topic length width height mass z_offset min_range max_range mesh">
     <!-- z_offset: distance between base plate and laser center (= center of mesh) -->
     <link name="${name}_mount_link">
