Commit message: Add new macros for more accurate Gazebo specification of specific TiM models

File: urdf/sick_scan.urdf.xacro (robot description, xacro)
@@ -7,5 +7,17 @@
     <xacro:sick_tim name="${name}" ros_topic="${ros_topic}"
       length="0.06" width="0.06" height="0.079" mass="0.150" z_offset="0.05595"
-      min_range="0.05" max_range="4.0"
+      min_range="0.05" max_range="4.0" samples="271"
+      mesh="package://sick_scan/meshes/sick_tim_5xx.stl" />
+  </xacro:macro>
+  <xacro:macro name="sick_tim_56x" params="name ros_topic">
+    <xacro:sick_tim name="${name}" ros_topic="${ros_topic}"
+      length="0.06" width="0.06" height="0.079" mass="0.150" z_offset="0.05595"
+      min_range="0.05" max_range="10.0" samples="811"
+      mesh="package://sick_scan/meshes/sick_tim_5xx.stl" />
+  </xacro:macro>
+  <xacro:macro name="sick_tim_57x" params="name ros_topic">
+    <xacro:sick_tim name="${name}" ros_topic="${ros_topic}"
+      length="0.06" width="0.06" height="0.079" mass="0.150" z_offset="0.05595"
+      min_range="0.05" max_range="25.0" samples="811"
       mesh="package://sick_scan/meshes/sick_tim_5xx.stl" />
   </xacro:macro>
@@ -13,8 +25,8 @@
     <xacro:sick_tim name="${name}" ros_topic="${ros_topic}"
       length="0.06" width="0.06" height="0.079" mass="0.150" z_offset="0.05595"
-      min_range="0.05" max_range="4.0"
+      min_range="0.05" max_range="4.0" samples="271"
       mesh="package://sick_scan/meshes/sick_tim_5xx.stl" />
   </xacro:macro>
-  <xacro:macro name="sick_tim" params="name ros_topic length width height mass z_offset min_range max_range mesh">
+  <xacro:macro name="sick_tim" params="name ros_topic length width height mass z_offset min_range max_range samples mesh">
     <!-- z_offset: distance between base plate and laser center (= center of mesh) -->
     <link name="${name}_mount_link">
@@ -66,5 +78,5 @@
           <scan>
             <horizontal>
-              <samples>271</samples>
+              <samples>${samples}</samples>
               <resolution>1</resolution>
               <min_angle>${min_angle}</min_angle>

Commit message: Add option to specify angle limits to gazebo configuration

File: urdf/sick_scan.urdf.xacro (robot description, xacro)
@@ -10,13 +10,15 @@
       mesh="package://sick_scan/meshes/sick_tim_5xx.stl" />
   </xacro:macro>
-  <xacro:macro name="sick_tim_56x" params="name ros_topic">
+  <xacro:macro name="sick_tim_56x" params="name ros_topic min_angle:=-2.357 max_angle:=2.357">
     <xacro:sick_tim name="${name}" ros_topic="${ros_topic}"
       length="0.06" width="0.06" height="0.079" mass="0.150" z_offset="0.05595"
+      min_angle="${min_angle}" max_angle="${max_angle}"
       min_range="0.05" max_range="10.0" samples="811"
       mesh="package://sick_scan/meshes/sick_tim_5xx.stl" />
   </xacro:macro>
-  <xacro:macro name="sick_tim_57x" params="name ros_topic">
+  <xacro:macro name="sick_tim_57x" params="name ros_topic min_angle:=-2.357 max_angle:=2.357">
     <xacro:sick_tim name="${name}" ros_topic="${ros_topic}"
       length="0.06" width="0.06" height="0.079" mass="0.150" z_offset="0.05595"
+      min_angle="${min_angle}" max_angle="${max_angle}"
       min_range="0.05" max_range="25.0" samples="811"
       mesh="package://sick_scan/meshes/sick_tim_5xx.stl" />
@@ -28,5 +30,5 @@
       mesh="package://sick_scan/meshes/sick_tim_5xx.stl" />
   </xacro:macro>
-  <xacro:macro name="sick_tim" params="name ros_topic length width height mass z_offset min_range max_range samples mesh">
+  <xacro:macro name="sick_tim" params="name ros_topic length width height mass z_offset min_angle max_angle min_range max_range samples mesh">
     <!-- z_offset: distance between base plate and laser center (= center of mesh) -->
     <link name="${name}_mount_link">
@@ -65,7 +67,7 @@
       </inertial>
     </link>
-    <xacro:sick_tim_laser_gazebo_v0 name="${name}" link="${name}" ros_topic="${ros_topic}" update_rate="15.0" min_angle="-2.357" max_angle="2.357" min_range="${min_range}" max_range="${max_range}"/>
+    <xacro:sick_tim_laser_gazebo_v0 name="${name}" link="${name}" ros_topic="${ros_topic}" update_rate="15.0" min_angle="-2.357" max_angle="2.357" min_range="${min_range}" max_range="${max_range}" samples="${samples}"/>
   </xacro:macro>
-  <xacro:macro name="sick_tim_laser_gazebo_v0" params="name link ros_topic update_rate min_angle max_angle min_range max_range">
+  <xacro:macro name="sick_tim_laser_gazebo_v0" params="name link ros_topic update_rate min_angle max_angle min_range max_range samples">
     <gazebo reference="${link}">
       <material value="Gazebo/Blue" />

Commit message: Add samples param to the macro

File: urdf/sick_scan.urdf.xacro (robot description, xacro)
@@ -10,16 +10,16 @@
       mesh="package://sick_scan/meshes/sick_tim_5xx.stl" />
   </xacro:macro>
-  <xacro:macro name="sick_tim_56x" params="name ros_topic min_angle:=-2.357 max_angle:=2.357">
+  <xacro:macro name="sick_tim_56x" params="name ros_topic min_angle:=-2.357 max_angle:=2.357 samples:=811">
     <xacro:sick_tim name="${name}" ros_topic="${ros_topic}"
       length="0.06" width="0.06" height="0.079" mass="0.150" z_offset="0.05595"
       min_angle="${min_angle}" max_angle="${max_angle}"
-      min_range="0.05" max_range="10.0" samples="811"
+      min_range="0.05" max_range="10.0" samples="${samples}"
       mesh="package://sick_scan/meshes/sick_tim_5xx.stl" />
   </xacro:macro>
-  <xacro:macro name="sick_tim_57x" params="name ros_topic min_angle:=-2.357 max_angle:=2.357">
+  <xacro:macro name="sick_tim_57x" params="name ros_topic min_angle:=-2.357 max_angle:=2.357 samples:=811">
     <xacro:sick_tim name="${name}" ros_topic="${ros_topic}"
       length="0.06" width="0.06" height="0.079" mass="0.150" z_offset="0.05595"
       min_angle="${min_angle}" max_angle="${max_angle}"
-      min_range="0.05" max_range="25.0" samples="811"
+      min_range="0.05" max_range="25.0" samples="${samples}"
       mesh="package://sick_scan/meshes/sick_tim_5xx.stl" />
   </xacro:macro>
