Commit message: Fix Gazebo noise configuration, and add configurable noise parameter to Xacro macros.

File: urdf/sick_lms1xx.urdf.xacro (robot description, xacro)
@@ -4,10 +4,10 @@
   xmlns:sensor="http://playerstage.sourceforge.net/gazebo/xmlschema/#sensor"
   xmlns:xacro="http://ros.org/wiki/xacro">
-  <xacro:macro name="sick_lms_1xx" params="name ros_topic">
+  <xacro:macro name="sick_lms_1xx" params="name ros_topic gaussian_noise:=0.006">
     <xacro:sick_lms_1 name="${name}" ros_topic="${ros_topic}"
       length="0.105636" width="0.102301" height="0.161782" mass="1.1" x_offset="0.052811" z_offset="-0.008195"
-      min_range="0.5" max_range="20.0"/>
+      min_range="0.5" max_range="20.0" gaussian_noise="${gaussian_noise}" />
   </xacro:macro>
-  <xacro:macro name="sick_lms_1" params="name ros_topic length width height mass x_offset z_offset min_range max_range">
+  <xacro:macro name="sick_lms_1" params="name ros_topic length width height mass x_offset z_offset min_range max_range gaussian_noise">
     <link name="${name}_mount_link">
       <visual>
@@ -45,7 +45,7 @@
       </inertial>
     </link>
-    <xacro:sick_lms_1_laser_gazebo_v0 name="${name}" link="${name}_laser" ros_topic="${ros_topic}" update_rate="15.0" min_angle="-2.357" max_angle="2.357" min_range="${min_range}" max_range="${max_range}"/>
+    <xacro:sick_lms_1_laser_gazebo_v0 name="${name}" link="${name}_laser" ros_topic="${ros_topic}" update_rate="15.0" min_angle="-2.357" max_angle="2.357" min_range="${min_range}" max_range="${max_range}" gaussian_noise="${gaussian_noise}" />
   </xacro:macro>
-  <xacro:macro name="sick_lms_1_laser_gazebo_v0" params="name link ros_topic update_rate min_angle max_angle min_range max_range">
+  <xacro:macro name="sick_lms_1_laser_gazebo_v0" params="name link ros_topic update_rate min_angle max_angle min_range max_range gaussian_noise">
     <gazebo reference="${link}">
       <material value="Gazebo/Blue" />
@@ -69,9 +69,11 @@
             <resolution>0.01</resolution>
           </range>
+          <noise>
+            <type>gaussian</type>
+            <mean>0.0</mean>
+            <stddev>${gaussian_noise}</stddev>
+          </noise>
         </ray>
         <plugin name="gazebo_ros_${name}_controller" filename="libgazebo_ros_laser.so">
-          <gaussianNoise>0.005</gaussianNoise>
-          <alwaysOn>true</alwaysOn>
-          <updateRate>${update_rate}</updateRate>
           <topicName>${ros_topic}</topicName>
           <frameName>${link}</frameName>

File: urdf/sick_lms5xx.urdf.xacro (robot description, xacro)
@@ -4,10 +4,10 @@
   xmlns:sensor="http://playerstage.sourceforge.net/gazebo/xmlschema/#sensor"
   xmlns:xacro="http://ros.org/wiki/xacro">
-  <xacro:macro name="sick_lms_5xx" params="name ros_topic">
+  <xacro:macro name="sick_lms_5xx" params="name ros_topic gaussian_noise:=0.004">
     <xacro:sick_lms_5 name="${name}" ros_topic="${ros_topic}"
       length="0.159277" width="0.155002" height="0.196397" mass="3.7" x_offset="0.079205" z_offset="-0.053449"
-      min_range="1.0" max_range="80.0"/>
+      min_range="1.0" max_range="80.0" gaussian_noise="${gaussian_noise}" />
   </xacro:macro>
-  <xacro:macro name="sick_lms_5" params="name ros_topic length width height mass x_offset z_offset min_range max_range">
+  <xacro:macro name="sick_lms_5" params="name ros_topic length width height mass x_offset z_offset min_range max_range gaussian_noise">
     <link name="${name}_mount_link">
       <visual>
@@ -45,7 +45,7 @@
       </inertial>
     </link>
-    <xacro:sick_lms_5_laser_gazebo_v0 name="${name}" link="${name}_laser" ros_topic="${ros_topic}" update_rate="50.0" min_angle="-1.65806" max_angle="1.65806" min_range="${min_range}" max_range="${max_range}"/>
+    <xacro:sick_lms_5_laser_gazebo_v0 name="${name}" link="${name}_laser" ros_topic="${ros_topic}" update_rate="50.0" min_angle="-1.65806" max_angle="1.65806" min_range="${min_range}" max_range="${max_range}" gaussian_noise="${gaussian_noise}" />
   </xacro:macro>
-  <xacro:macro name="sick_lms_5_laser_gazebo_v0" params="name link ros_topic update_rate min_angle max_angle min_range max_range">
+  <xacro:macro name="sick_lms_5_laser_gazebo_v0" params="name link ros_topic update_rate min_angle max_angle min_range max_range gaussian_noise">
     <gazebo reference="${link}">
       <material value="Gazebo/Blue" />
@@ -69,9 +69,11 @@
             <resolution>0.01</resolution>
           </range>
+          <noise>
+            <type>gaussian</type>
+            <mean>0.0</mean>
+            <stddev>${gaussian_noise}</stddev>
+          </noise>
         </ray>
         <plugin name="gazebo_ros_${name}_controller" filename="libgazebo_ros_laser.so">
-          <gaussianNoise>0.005</gaussianNoise>
-          <alwaysOn>true</alwaysOn>
-          <updateRate>${update_rate}</updateRate>
           <topicName>${ros_topic}</topicName>
           <frameName>${link}</frameName>

File: urdf/sick_scan.urdf.xacro (robot description, xacro)
@@ -4,33 +4,33 @@
   xmlns:sensor="http://playerstage.sourceforge.net/gazebo/xmlschema/#sensor"
   xmlns:xacro="http://ros.org/wiki/xacro">
-  <xacro:macro name="sick_tim_5xx" params="name ros_topic min_angle:=-2.357 max_angle:=2.357 samples:=271">
+  <xacro:macro name="sick_tim_5xx" params="name ros_topic min_angle:=-2.357 max_angle:=2.357 gaussian_noise:=0.01 samples:=271">
     <xacro:sick_tim name="${name}" ros_topic="${ros_topic}"
       length="0.06" width="0.06" height="0.079" mass="0.150" z_offset="0.05595"
       min_angle="${min_angle}" max_angle="${max_angle}"
-      min_range="0.05" max_range="4.0" samples="${samples}"
+      min_range="0.05" max_range="4.0" gaussian_noise="${gaussian_noise}" samples="${samples}"
       mesh="package://sick_scan/meshes/sick_tim_5xx.stl" />
   </xacro:macro>
-  <xacro:macro name="sick_tim_56x" params="name ros_topic min_angle:=-2.357 max_angle:=2.357 samples:=811">
+  <xacro:macro name="sick_tim_56x" params="name ros_topic min_angle:=-2.357 max_angle:=2.357 gaussian_noise:=0.01 samples:=811">
     <xacro:sick_tim name="${name}" ros_topic="${ros_topic}"
       length="0.06" width="0.06" height="0.079" mass="0.150" z_offset="0.05595"
       min_angle="${min_angle}" max_angle="${max_angle}"
-      min_range="0.05" max_range="10.0" samples="${samples}"
+      min_range="0.05" max_range="10.0" gaussian_noise="${gaussian_noise}" samples="${samples}"
       mesh="package://sick_scan/meshes/sick_tim_5xx.stl" />
   </xacro:macro>
-  <xacro:macro name="sick_tim_57x" params="name ros_topic min_angle:=-2.357 max_angle:=2.357 samples:=811">
+  <xacro:macro name="sick_tim_57x" params="name ros_topic min_angle:=-2.357 max_angle:=2.357 gaussian_noise:=0.01 samples:=811">
     <xacro:sick_tim name="${name}" ros_topic="${ros_topic}"
       length="0.06" width="0.06" height="0.079" mass="0.150" z_offset="0.05595"
       min_angle="${min_angle}" max_angle="${max_angle}"
-      min_range="0.05" max_range="25.0" samples="${samples}"
+      min_range="0.05" max_range="25.0" gaussian_noise="${gaussian_noise}" samples="${samples}"
       mesh="package://sick_scan/meshes/sick_tim_5xx.stl" />
   </xacro:macro>
-  <xacro:macro name="sick_mrs_1xxx" params="name ros_topic min_angle:=-2.357 max_angle:=2.357 samples:=271">
+  <xacro:macro name="sick_mrs_1xxx" params="name ros_topic min_angle:=-2.357 max_angle:=2.357 gaussian_noise:=0.015 samples:=271">
     <xacro:sick_tim name="${name}" ros_topic="${ros_topic}"
       length="0.06" width="0.06" height="0.079" mass="0.150" z_offset="0.05595"
       min_angle="${min_angle}" max_angle="${max_angle}"
-      min_range="0.05" max_range="4.0" samples="${samples}"
+      min_range="0.05" max_range="4.0" gaussian_noise="${gaussian_noise}" samples="${samples}"
       mesh="package://sick_scan/meshes/sick_tim_5xx.stl" />
   </xacro:macro>
-  <xacro:macro name="sick_tim" params="name ros_topic length width height mass z_offset min_angle max_angle min_range max_range samples mesh">
+  <xacro:macro name="sick_tim" params="name ros_topic length width height mass z_offset min_angle max_angle min_range max_range gaussian_noise samples mesh">
     <!-- z_offset: distance between base plate and laser center (= center of mesh) -->
     <link name="${name}_mount_link">
@@ -69,7 +69,7 @@
       </inertial>
     </link>
-    <xacro:sick_tim_laser_gazebo_v0 name="${name}" link="${name}" ros_topic="${ros_topic}" update_rate="15.0" min_angle="${min_angle}" max_angle="${max_angle}" min_range="${min_range}" max_range="${max_range}" samples="${samples}"/>
+    <xacro:sick_tim_laser_gazebo_v0 name="${name}" link="${name}" ros_topic="${ros_topic}" update_rate="15.0" min_angle="${min_angle}" max_angle="${max_angle}" min_range="${min_range}" max_range="${max_range}" gaussian_noise="${gaussian_noise}" samples="${samples}" />
   </xacro:macro>
-  <xacro:macro name="sick_tim_laser_gazebo_v0" params="name link ros_topic update_rate min_angle max_angle min_range max_range samples">
+  <xacro:macro name="sick_tim_laser_gazebo_v0" params="name link ros_topic update_rate min_angle max_angle min_range max_range gaussian_noise samples">
     <gazebo reference="${link}">
       <material value="Gazebo/Blue" />
@@ -93,9 +93,11 @@
             <resolution>0.01</resolution>
           </range>
+          <noise>
+            <type>gaussian</type>
+            <mean>0.0</mean>
+            <stddev>${gaussian_noise}</stddev>
+          </noise>
         </ray>
         <plugin name="gazebo_ros_${name}_controller" filename="libgazebo_ros_laser.so">
-          <gaussianNoise>0.005</gaussianNoise>
-          <alwaysOn>true</alwaysOn>
-          <updateRate>${update_rate}</updateRate>
           <topicName>${ros_topic}</topicName>
           <frameName>${link}</frameName>
